File: hardware/turtle/turtle.kicad_sch (KiCad schematic)
At the start: 34 parts, among them J1 Motor Left, J2 Motor Right, J3 Battery, M1 Motor_Servo, Q1 BP103B, Q2 BP103B, SW1 SW_Push, SW2 SW_Wuerth_450301014042, U1 PicoW, U2 ULN2803A

Commit message: Update for ordered components.
ULN2803A instead of ULN2803C.
Speaker with 5mm pitch.
Parts:
- removed U2: ULN2803A, Package_SO:SOIC-20W_7.5x12.8mm_P1.27mm, symbol uln2803c:ULN2803C
- added U2: ULN2803A, Package_SO:SOIC-18W_7.5x11.6mm_P1.27mm, symbol Transistor_Array:ULN2803A
- LS1: footprint Buzzer_Beeper:Buzzer_12x9.5RM7.6 -> Buzzer_Beeper:Buzzer_TDK_PS1240P02BT_D12.2mm_H6.5mm
- Q1, Q2: footprint LED_THT:LED_D5.0mm_Clear -> library:LED_D5.0mm_Horizontal_O1.27mm_Z3.0mm_truncated_silkscreen
Connections:
- net GNDD: now also U2.9 (GND)
- net Motor Left A: now also U2.8 (I8)
- net Motor Left B: now also U2.7 (I7)
- net Motor Left C: now also U2.6 (I6)
- net Motor Left D: now also U2.5 (I5)
- net Motor Right A: now also U2.4 (I4)
- net Motor Right B: now also U2.3 (I3)
- net Motor Right C: now also U2.2 (I2)
- net Motor Right D: now also U2.1 (I1)
- net VBat: now also U2.10 (COM)
- net at J2.2 (Pin_2): now also U2.15 (O4)
- net at J2.3 (Pin_3): now also U2.16 (O3)
- net at J2.4 (Pin_4): now also U2.17 (O2)
- net at J2.5 (Pin_5): now also U2.18 (O1)
- net at J1.2 (Pin_2): now also U2.11 (O8)
- net at J1.3 (Pin_3): now also U2.12 (O7)
- net at J1.4 (Pin_4): now also U2.13 (O6)
- net at J1.5 (Pin_5): now also U2.14 (O5)
Changed lines of the file:
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@@
 			)
 		)
-		(property "Footprint" "LED_THT:LED_D5.0mm_Clear"
+		(property "Footprint" "library:LED_D5.0mm_Horizontal_O1.27mm_Z3.0mm_truncated_silkscreen"
 			(at 206.502 157.226 0)
 			(effects
@@
 	)
 	(symbol
+		(lib_id "Transistor_Array:ULN2803A")
+		(at 133.35 69.85 0)
+		(unit 1)
+		(exclude_from_sim no)
+		(in_bom yes)
+		(on_board yes)
+		(dnp no)
+		(fields_autoplaced yes)
+		(property "Reference" "U2"
+			(at 133.35 54.61 0)
+			(effects
+				(font
+					(size 1.27 1.27)
+				)
+			)
+		)
+		(property "Value" "ULN2803A"
+			(at 133.35 57.15 0)
+			(effects
+				(font
+					(size 1.27 1.27)
+				)
+			)
+		)
+		(property "Footprint" "Package_SO:SOIC-18W_7.5x11.6mm_P1.27mm"
+			(at 134.62 86.36 0)
+			(effects
+				(font
+					(size 1.27 1.27)
+				)
+				(justify left)
+				(hide yes)
+			)
+		)
+		(property "Datasheet" "http://www.ti.com/lit/ds/symlink/uln2803a.pdf"
+			(at 135.89 74.93 0)
+			(effects
+				(font
+					(size 1.27 1.27)
+				)
+				(hide yes)
+			)
+		)
+		(property "Description" "Darlington Transistor Arrays, SOIC18/DIP18"
+			(at 133.35 69.85 0)
+			(effects
+				(font
+					(size 1.27 1.27)
+				)
+				(hide yes)
+			)
+		)
+		(pin "1"
+		)
+		(pin "17"
+		)
+		(pin "7"
+		)
+		(pin "16"
+		)
+		(pin "3"
+		)
+		(pin "6"
+		)
+		(pin "5"
+		)
+		(pin "14"
+		)
+		(pin "18"
+		)
+		(pin "8"
+		)
+		(pin "13"
+		)
+		(pin "12"
+		)
+		(pin "11"
+		)
+		(pin "10"
+		)
+		(pin "15"
+		)
+		(pin "2"
+		)
+		(pin "4"
+		)
+		(pin "9"
+		)
+		(instances
+			(project ""
+				(path "/46da222e-9eeb-478a-b929-a85b6b040af6"
+					(reference "U2")
+					(unit 1)
+				)
+			)
+		)
+	)
+	(symbol
 		(lib_id "power:+3.3V")
 		(at 120.65 114.3 0)
@@
 	)
 	(symbol
-		(lib_id "uln2803c:ULN2803C")
-		(at 133.35 69.85 0)
-		(unit 1)
-		(exclude_from_sim no)
-		(in_bom yes)
-		(on_board yes)
-		(dnp no)
-		(property "Reference" "U2"
-			(at 133.35 54.61 0)
-			(effects
-				(font
-					(size 1.27 1.27)
-				)
-			)
-		)
-		(property "Value" "ULN2803A"
-			(at 133.35 57.15 0)
-			(effects
-				(font
-					(size 1.27 1.27)
-				)
-			)
-		)
-		(property "Footprint" "Package_SO:SOIC-20W_7.5x12.8mm_P1.27mm"
-			(at 134.62 86.36 0)
-			(effects
-				(font
-					(size 1.27 1.27)
-				)
-				(justify left)
-				(hide yes)
-			)
-		)
-		(property "Datasheet" "https://www.ti.com/lit/ds/symlink/uln2803c.pdf"
-			(at 135.89 74.93 0)
-			(effects
-				(font
-					(size 1.27 1.27)
-				)
-				(hide yes)
-			)
-		)
-		(property "Description" "Darlington Transistor Arrays, SOIC20"
-			(at 133.35 69.85 0)
-			(effects
-				(font
-					(size 1.27 1.27)
-				)
-				(hide yes)
-			)
-		)
-		(pin "16"
-		)
-		(pin "15"
-		)
-		(pin "11"
-		)
-		(pin "2"
-		)
-		(pin "17"
-		)
-		(pin "10"
-		)
-		(pin "6"
-		)
-		(pin "3"
-		)
-		(pin "4"
-		)
-		(pin "14"
-		)
-		(pin "1"
-		)
-		(pin "9"
-		)
-		(pin "7"
-		)
-		(pin "8"
-		)
-		(pin "5"
-		)
-		(pin "18"
-		)
-		(pin "12"
-		)
-		(pin "13"
-		)
-		(pin "20"
-		)
-		(pin "19"
-		)
-		(instances
-			(project ""
-				(path "/46da222e-9eeb-478a-b929-a85b6b040af6"
-					(reference "U2")
-					(unit 1)
-				)
-			)
-		)
-	)
-	(symbol
 		(lib_id "Sensor_Optical:BP103B")
 		(at 118.11 153.67 0)
@@
 			)
 		)
-		(property "Footprint" "LED_THT:LED_D5.0mm_Clear"
+		(property "Footprint" "library:LED_D5.0mm_Horizontal_O1.27mm_Z3.0mm_truncated_silkscreen"
 			(at 130.302 157.226 0)
 			(effects
@@
 			)
 		)
-		(property "Footprint" "Buzzer_Beeper:Buzzer_12x9.5RM7.6"
+		(property "Footprint" "Buzzer_Beeper:Buzzer_TDK_PS1240P02BT_D12.2mm_H6.5mm"
 			(at 56.261 114.3 0)
 			(effects
