File: hardware/turtle/turtle.kicad_pcb (KiCad board)
At the start: 2 copper layers, 52 x 48 mm, 34 parts, among them J1 Motor Left, J2 Motor Right, J3 Battery, M1 Motor_Servo, Q1 BP103B, Q2 BP103B, SW1 SW_Push, SW2 SW_Wuerth_450301014042, U1 PicoW, U2 ULN2803A

Commit message: Update for ordered components.
ULN2803A instead of ULN2803C.
Speaker with 5mm pitch.
Parts:
- LS1: footprint Buzzer_Beeper:Buzzer_12x9.5RM7.6 -> Buzzer_Beeper:Buzzer_TDK_PS1240P02BT_D12.2mm_H6.5mm
- U2: footprint Package_SO:SOIC-20W_7.5x12.8mm_P1.27mm -> Package_SO:SOIC-18W_7.5x11.6mm_P1.27mm
- moved LS1 1.43 mm to (150.0, 118.4)
- moved R9 0.91 mm to (152.4, 117.5), turned to -90 degrees
- moved U2 0.64 mm to (151.8, 101.6)
Connections:
- U2 pad 10: unconnected-(U2-NC-Pad10) -> VBat
- U2 pad 11: unconnected-(U2-NC-Pad11) -> Net-(J1-Pin_2)
- U2 pad 12: VBat -> Net-(J1-Pin_3)
- U2 pad 13: Net-(J1-Pin_2) -> Net-(J1-Pin_4)
- U2 pad 14: Net-(J1-Pin_3) -> Net-(J1-Pin_5)
- U2 pad 15: Net-(J1-Pin_4) -> Net-(J2-Pin_2)
- U2 pad 16: Net-(J1-Pin_5) -> Net-(J2-Pin_3)
- U2 pad 17: Net-(J2-Pin_2) -> Net-(J2-Pin_4)
- U2 pad 18: Net-(J2-Pin_3) -> Net-(J2-Pin_5)
Routing:
- net /Speaker: track 32.9 -> 35.4 mm
- net Net-(LS1-Pad1): track 2.89 -> 2.37 mm

Commit message: Add logo and revision to PCB.
Parts:
- added REF**: LOGO, Logo:LogoS7_5mm, F.Cu at (135.1, 115.3)
Other:
- board text added: "Turtle r1"
